Commit message: Added IMU and LIDAR

File: dingo_description/urdf/dingo-d.urdf.xacro (robot description, xacro)
@@ -215,4 +215,29 @@
     <child link="front_bumper_mount" />
   </joint>
+  <!-- LIDAR -->
+  <link name="base_scan">
+    <inertial>
+      <mass value="0.001"/>
+      <origin xyz="0 0 0" rpy="0 0 0"/>
+      <inertia ixx="${dummy_inertia}" ixy="0.0" ixz="0.0" iyy="${dummy_inertia}" iyz="0.0" izz="${dummy_inertia}"/>
+    </inertial>
+    <visual>
+      <origin xyz="0 0 0" rpy="0 0 0"/>
+      <geometry>
+        <cylinder radius="0.041" length="0.076"/>
+      </geometry>
+    </visual>
+    <collision>
+      <origin xyz="0 0 0" rpy="0 0 0"/>
+      <geometry>
+        <cylinder radius="0.041" length="0.076"/>
+      </geometry>
+    </collision>
+  </link>
+  <joint name="lidar_joint" type="fixed">
+    <parent link="chassis_link"/>
+    <child link="base_scan" />
+    <origin xyz="0.0 0.0 0.15" rpy="0 0 0" />
+  </joint>
   <!-- Bring in simulation data for Gazebo. -->
   <xacro:include filename="$(find dingo_description)/urdf/dingo.gazebo" />

Commit message: working dingo navigation with gazebo sim

File: dingo_description/urdf/dingo-d.urdf.xacro (robot description, xacro)
@@ -115,4 +115,10 @@
     <implicitSpringDamper>1</implicitSpringDamper>
   </gazebo>
+  <link name="base_footprint"/>
+  <joint name="base_joint" type="fixed">
+    <parent link="base_footprint"/>
+    <child link="base_link"/>
+    <origin xyz="0.0 0.0 0.010" rpy="0 0 0"/>
+  </joint>
   <link name="base_link"></link>
   <joint name="base_link_joint" type="fixed">
